File: projects/garden_guard/garden_guard.kicad_sch (KiCad schematic)
At the start: 8 parts

Commit message: - Find part numbers for CM5 parts - Minor CM5 symbol, footprint adjustments - Move to uniform small resistor and capacitor symbols - Add *lck to .gitignore
Other:
- sheet CM5_HighSpeed ports: added PWR_SRC_ST; removed PWR_SRC_SEL
- sheet Power ports: added PWR_SRC_ST; removed PWR_SRC_SEL
- note removed: "Connectors ------- CSI/DSI 0 CSI/DSI 1"
Changed lines of the file:
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@@
 	(generator_version "9.0")
 	(paper "A4")
-	(text "Connectors\n-------\nCSI/DSI 0\nCSI/DSI 1"
-		(exclude_from_sim no)
-		(at 177.8 24.13 0)
-		(effects
-			(font
-				(size 1.27 1.27)
-			)
-			(justify left bottom)
-		)
-	)
 	(text "Features\n-------\n12V -> 5V Buck\nINA226 Current Sensor (5V bus)\nINA226 Current Sensor (3V3 bus, if not measured\ninternally)\nDS18b20 Temperature Sensor Header (SSD)\nDS18b20 Temperature Sensor Header (Enclosure)\nPoE (???)\nIR LED Power (possible via 5V USB-C?)\nIR LED FET\nINA226 Current Sensor (IR LED out)"
 		(exclude_from_sim no)
@@
 	)
 	(symbol
+		(lib_name "MountingHole_5")
 		(lib_id "Mechanical:MountingHole")
 		(at 16.51 194.31 0)
@@
 	)
 	(symbol
+		(lib_name "MountingHole_4")
 		(lib_id "Mechanical:MountingHole")
 		(at 16.51 189.23 0)
@@
 	)
 	(symbol
+		(lib_name "MountingHole_1")
 		(lib_id "Mechanical:MountingHole")
 		(at 16.51 179.07 0)
@@
 	)
 	(symbol
+		(lib_name "MountingHole_3")
 		(lib_id "Mechanical:MountingHole")
 		(at 37.465 179.07 0)
@@
 	)
 	(symbol
+		(lib_name "MountingHole_7")
 		(lib_id "Mechanical:MountingHole")
 		(at 37.465 194.31 0)
@@
 	)
 	(symbol
+		(lib_name "MountingHole_2")
 		(lib_id "Mechanical:MountingHole")
 		(at 37.465 189.23 0)
@@
 	)
 	(symbol
+		(lib_name "MountingHole_6")
 		(lib_id "Mechanical:MountingHole")
 		(at 37.465 184.15 0)
@@
 			)
 		)
-		(pin "PWR_SRC_SEL" input
+		(pin "PWR_SRC_ST" input
 			(at 125.73 151.13 180)
 			(effects
@@
 			)
 		)
-		(pin "PWR_SRC_SEL" output
+		(pin "PWR_SRC_ST" output
 			(at 96.52 151.13 0)
 			(effects

Commit message: - Add M.2 power and connector layout - Add micro HDMI to schematic and layout - Add microSD layout - Add IR illuminator and solenoid output MOSFET layouts - Add USB-C layout
Other:
- sheet CM5_GPIO (Ethernet, GPIO, MicroSD) ports: added +5v; removed none
Changed lines of the file:
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@@
+	(wire
+		(pts
+			(xy 119.38 46.99) (xy 125.73 46.99)
+		)
+		(stroke
+			(width 0)
+			(type default)
+		)
+	)
 	(wire
 		(pts
@@
 	(label "+12v"
 		(at 203.2 119.38 0)
+		(effects
+			(font
+				(size 1.27 1.27)
+			)
+			(justify left bottom)
+		)
+	)
+	(label "+5v"
+		(at 119.38 46.99 0)
 		(effects
 			(font
@@
 			(effects
 				(font
+					(size 1.27 1.27)
+				)
+				(justify left)
+			)
+		)
+		(pin "+5v" input
+			(at 125.73 46.99 180)
+			(effects
+				(font
