File: projects/garden_guard/garden_guard.kicad_sch (KiCad schematic)
At the start: 8 parts

Commit message: - All footprints laid out; DRC NOT run yet, likely has many violations - Thin out peripheral headers, move remaining to dispersed test pads - Update kicad-libraries
Parts:
- removed H5, H6, H7, H8: MountingHole, CM5IO:MountingHole_2.7mm_M2.5_DIN965, symbol Mechanical:MountingHole
