File: projects/garden_guard/CM5_GPIO.kicad_sch (KiCad schematic)
At the start: 10 parts, among them J12 Mini HDMI, J5 Conn_01x22_Female, J6 Conn_01x22_Female, U14 RT9742SNGV

Commit message: JLC part audit - CM5_HighSpeed - CM5_GPIO - PCIe_M2
Parts:
- C31, C32: footprint Resistor_SMD:R_0603_1608Metric -> Capacitor_SMD:C_0603_1608Metric; Class (none) -> capacitor; Critical (none) -> no; Dielectric_Class (none) -> X7R; JLCPCB_PN (none) -> C2167527; Package (none) -> 0603
- J12: Class (none) -> connector; Critical (none) -> yes; JLCPCB_PN (none) -> C573682; MPN (none) -> 2013978-2; Mfr (none) -> TE Connectivity
- J5, J6: Class (none) -> connector; Critical (none) -> yes; JLCPCB_PN (none) -> C2906120
- Module1: Class (none) -> cpu; Critical (none) -> yes; JLCPCB_PN (none) -> C7435219
- R10, R11, R9: footprint Capacitor_SMD:C_0603_1608Metric -> Resistor_SMD:R_0603_1608Metric; Class (none) -> resistor; Critical (none) -> no; JLCPCB_PN (none) -> C844925; Mfr Vishay Dale -> Vishay; Package (none) -> 0603; Power 1/8W -> 1/10W; Tolerance (none) -> 1%; Voltage (none) -> 75V
- U14: Class (none) -> load_switch; Critical (none) -> review; JLCPCB_PN (none) -> C3235509; Package (none) -> SOT-23-3

Commit message: - All footprints laid out; DRC NOT run yet, likely has many violations - Thin out peripheral headers, move remaining to dispersed test pads - Update kicad-libraries
Connections:
- net USBOTG_ID: no longer names the net of Module1.101 (USB_OTG_ID)
- no-connect marks 27 -> 28
Changed lines of the file:
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@@
+	)
+	(no_connect
+		(at 100.33 27.94)
 	)
 	(no_connect
@@
 			(width 0)
 			(type default)
-		)
-	)
-	(wire
-		(pts
-			(xy 106.68 27.94) (xy 100.33 27.94)
-		)
-		(stroke
-			(width 0)
-			(type solid)
 		)
 	)
@@
 		(effects
 			(font
-				(size 1.27 1.27)
-			)
-			(justify left)
-		)
-	)
-	(hierarchical_label "USBOTG_ID"
-		(shape input)
-		(at 106.68 27.94 0)
-		(effects
-			(font
