File: projects/garden_guard/CM5_HighSpeed.kicad_sch (KiCad schematic)
At the start: 28 parts, among them J1 Conn_02x07_Odd_Even, J2 Conn_01x03, J3 BM04B-SRSS-TB, J4 Micro_SD_Card_Det, SW1 Tact button, U1 SN74LVC1G07DBVR, U2 TPD4EUSB30, U3 TPD4EUSB30, U4 RT9742GGJ5, U5 MagJack-A70-112-331N126

Commit message: JLC part audit - CM5_HighSpeed - CM5_GPIO - PCIe_M2
Parts:
- removed C1: 10uF, Capacitor_SMD:C_0805_2012Metric, symbol Device:C
- added C1: 10uF, Capacitor_SMD:C_0805_2012Metric, symbol Device:C_Small
- BT1: Class (none) -> battery_holder; Critical (none) -> no; JLCPCB_PN (none) -> C5199422
- C2: footprint Resistor_SMD:R_0603_1608Metric -> Capacitor_SMD:C_0603_1608Metric; Class (none) -> capacitor; Critical (none) -> no; Dielectric_Class (none) -> X7R; JLCPCB_PN (none) -> C2167527; Mfr (none) -> KEMET; Package (none) -> 0603
- D1: Class (none) -> led; Color (none) -> green; Critical (none) -> no; JLCPCB_PN (none) -> C125113; Part Description Green 572nm LED Indication - Discrete 2.2V 2-SMD, No Lead -> Green 572nm LED Indication - Discrete 2.2V 2-SMD, No Lead
- D2: Class (none) -> led; Color (none) -> green; Critical (none) -> no; Field4 Digikey -> (none); JLCPCB_PN (none) -> C125113
- J3: Class (none) -> connector; Critical (none) -> yes; JLCPCB_PN (none) -> C160390; MPN (none) -> BM04B-SRSS-TB; Mfr (none) -> JST; Package (none) -> SMD,P=1mm
- J4: Class (none) -> connector; Critical (none) -> review; JLCPCB_PN (none) -> C428492
- Module1: Class (none) -> cpu; Critical (none) -> yes; JLCPCB_PN (none) -> C7435219
- R1, R5: Class (none) -> resistor; Critical (none) -> no; JLCPCB_PN (none) -> C844920; Mfr Vishay Dale -> Vishay; Package (none) -> 0603; Power (none) -> 1/10W; Tolerance (none) -> 1%; Voltage (none) -> 75V
- R2, R8: Class (none) -> resistor; Critical (none) -> no; JLCPCB_PN (none) -> C191124; MPN RC0603FR-0710KL -> ERJ3EKF1002V; Mfr YAGEO -> Panasonic; Package (none) -> 0603; Voltage (none) -> 75V
- R3: footprint Resistor_SMD:R_0603_1608Metric -> Resistor_SMD:R_0805_2012Metric; Class (none) -> resistor; Critical (none) -> no; JLCPCB_PN (none) -> C96345; Package (none) -> 0805; Power (none) -> 1/8W; Tolerance (none) -> 5%; Voltage (none) -> 150V
- R6, R7: Class (none) -> resistor; Critical (none) -> no; JLCPCB_PN (none) -> C844786; Mfr Vishay Dale -> Vishay; Package (none) -> 0603; Power 1/8W -> 1/10W; Voltage (none) -> 75V
- SW1: Class (none) -> button; Critical (none) -> no; JLCPCB_PN (none) -> C22462608
- U1: Class (none) -> logic_ic; Critical (none) -> review; JLCPCB_PN (none) -> C7829; Package (none) -> SOT-23-5
- U2, U3: Class (none) -> esd_protection; Critical (none) -> review; JLCPCB_PN (none) -> C90627; Package (none) -> USON-10(1x2.5)
- U4: Class (none) -> load_switch; Critical (none) -> review; JLCPCB_PN (none) -> C250547; Package (none) -> TSOT-23-5
- U5: Class (none) -> magjack; Critical (none) -> yes; JLCPCB_PN (none) -> C9900132877; MPN A60-112-331P4D2 -> A70-112-331N126; Mfr EDAC Inc. -> EDAC
Connections:
- net GND: now also C1.2
- net SD_PWR: now also C1.1

Commit message: - All footprints laid out; DRC NOT run yet, likely has many violations - Thin out peripheral headers, move remaining to dispersed test pads - Update kicad-libraries
Parts:
- removed J1: Conn_02x07_Odd_Even, Connector_PinHeader_2.54mm:PinHeader_2x07_P2.54mm_Vertical, symbol Connector_Generic:Conn_02x07_Odd_Even
- removed J2: Conn_01x03, Connector_PinHeader_2.54mm:PinHeader_1x03_P2.54mm_Vertical, symbol Connector_Generic:Conn_01x03
- removed SW1: Tact button, Button_Switch_THT:SW_Tactile_SPST_Angled_PTS645Vx58-2LFS, symbol Switch:SW_Push
- removed TP4: TestPoint, TestPoint:TestPoint_Pad_2.0x2.0mm, symbol Connector:TestPoint
- added J2: BM04B-SRSS-TB, Custom_Connector:BM04B-SRSS_JST, symbol Custom_Connector:BM04B-SRSS-TB
- added SW2: ~, Custom_Switch:PTS636_SK25F_SMTR_LFS, symbol Custom_Switch:PTS636_SK25F_SMTR_LFS
- TP1: value TestPoint -> BOOT; footprint TestPoint:TestPoint_Pad_2.0x2.0mm -> TestPoint:TestPoint_Pad_D1.0mm; Field4 nf -> (none); Field5 nf -> (none); Field6 nf -> (none); Field7 nf -> (none); Part Description Test point -> (none)
- TP2: value TestPoint -> PMIC; footprint TestPoint:TestPoint_Pad_2.0x2.0mm -> TestPoint:TestPoint_Pad_D1.0mm; Field4 nf -> (none); Field5 nf -> (none); Field6 nf -> (none); Field7 nf -> (none); Part Description Test point -> (none)
- TP3: value TestPoint -> PWR; footprint TestPoint:TestPoint_Pad_2.0x2.0mm -> TestPoint:TestPoint_Pad_D1.0mm; Field4 nf -> (none); Field5 nf -> (none); Field6 nf -> (none); Field7 nf -> (none); Part Description Test point -> (none)
Connections:
- net +5v: now also J2.1
- net FAN_PWM: no longer TP2.1
- net GND: now also J2.4, SW2.2
- net PMIC_ENABLE: now also TP2.1
- net PWR_BUT: now also TP3.1, SW2.1
- net TACHO: no longer TP3.1
- net UART0_RX: now also J2.3
- net UART0_TX: now also J2.2
- net nRPIBOOT: now also TP1.1
- net at D1.1 (K), R1.1: no longer TP1.1
- net BT_nDis: no longer names the net of Module1.91 (BT_nDisable)
- net EEPROM_nWP: no longer names the net of Module1.20 (EEPROM_nWP)
- net SYNC_OUT: no longer names the net of Module1.18 (Ethernet_SYNC_OUT(3.3v))
- net WL_nDis: no longer names the net of Module1.89 (WiFi_nDisable)
- no-connect marks 17 -> 21
Other:
- note added: "CM5 Test Points"
- note added: "Companion MCU"
- note added: "Connector for optional companion microcontroller"
- note added: "Jumper to GND nRPIBOOT: USB boot mode PWR_BUT: press to request power down, hold to force PMIC_EN: hard kill CM5 power rail"
- note added: "Pull-up added for Fans that don't have a strong internal pullup"
- note removed: "Force RPIBOOT = Jumper Pins 1-2"
- note removed: "Jumpers"
- note removed: "Not Fitted header"
- note removed: "R2 : Pullup added for Fans that don't have a strong internal pullup"
