File: projects/garden_guard/PCIe-M2.kicad_sch (KiCad schematic)
At the start: 21 parts, among them M1 M.2 Solder Nut, M2 M.2 Screw, U6 AP3441SHE-7B, U7 M.2 Socket, U8 ASEK-32.768KHZ-L-R-T

Commit message: JLC part audit - CM5_HighSpeed - CM5_GPIO - PCIe_M2
Parts:
- removed C3, C4: 10uF, Capacitor_SMD:C_0805_2012Metric, symbol Device:C_Small
- C10, C7, C8, C9: Class (none) -> capacitor; Critical (none) -> no; Dielectric_Class (none) -> X7R; JLCPCB_PN (none) -> C326595; MPN GRM21BR71A106KA73L -> CC0805KKX7R7BB106; Mfr Murata Electronics -> YAGEO; Package (none) -> 0805; Tolerance (none) -> 10%; Voltage (none) -> 16V
- C11: footprint Resistor_SMD:R_0603_1608Metric -> Capacitor_SMD:C_0603_1608Metric; Class (none) -> capacitor; Critical (none) -> no; Dielectric_Class (none) -> X7R; JLCPCB_PN (none) -> C2167527; Mfr (none) -> KEMET; Package (none) -> 0603
- C5: footprint Resistor_SMD:R_0603_1608Metric -> Capacitor_SMD:C_0603_1608Metric; Class (none) -> capacitor; Critical (none) -> no; Dielectric_Class (none) -> X7R; JLCPCB_PN (none) -> C2167527; Manufacturer KEMET -> (none); Mfr (none) -> KEMET; Package (none) -> 0603
- C6: footprint Resistor_SMD:R_0603_1608Metric -> Capacitor_SMD:C_0603_1608Metric; Class (none) -> capacitor; Critical (none) -> no; Dielectric (none) -> X7R; Dielectric_Class (none) -> X7R; JLCPCB_PN (none) -> C1621; MPN CC0603KRX7R8BB473 -> CL10B472KB8NNNC; Manufacturer YAGEO -> (none); Mfr (none) -> Samsung; Package (none) -> 0603; Part_Class (none) -> capacitor; Voltage 25V -> 50V
- D3: Class (none) -> led; Color (none) -> green; Critical (none) -> no; JLCPCB_PN (none) -> C125113
- L1: Class (none) -> inductor; Critical (none) -> review; JLCPCB_PN (none) -> C22404330; Package (none) -> SMD,5.7x5.2mm
- M1, M2: Critical (none) -> no; JLCPCB_PN (none) -> zNONE
- R12: Class (none) -> resistor; Critical (none) -> no; JLCPCB_PN (none) -> C14675; Package (none) -> 0603; Power (none) -> 1/10W; Voltage (none) -> 75V
- R13: Class (none) -> resistor; Critical (none) -> no; JLCPCB_PN (none) -> C191124; MPN RC0603FR-0710KL -> ERJ3EKF1002V; Mfr YAGEO -> Panasonic; Package (none) -> 0603; Voltage (none) -> 75V
- R14: Class (none) -> resistor; Critical (none) -> no; JLCPCB_PN (none) -> C844925; Mfr Vishay Dale -> Vishay; Package (none) -> 0603; Power 1/8W -> 1/10W; Tolerance (none) -> 1%; Voltage (none) -> 75V
- R15: Class (none) -> resistor; Critical (none) -> no; JLCPCB_PN (none) -> C844920; Mfr Vishay Dale -> Vishay; Package (none) -> 0603; Power (none) -> 1/10W; Tolerance (none) -> 1%; Voltage (none) -> 75V
- U6: Class (none) -> buck; Critical (none) -> review; JLCPCB_PN (none) -> C2070918
- U7: Class (none) -> connector; Critical (none) -> review; JLCPCB_PN (none) -> C590854; MPN MDT420M02003 -> 1-2199230-5; Mfr Amphenol -> TE Connectivity; Package (none) -> SMD,P=0.5mm
- U8: Class (none) -> crystal; Critical (none) -> review; Field7 abracon -> (none); JLCPCB_PN (none) -> C2650753; Package (none) -> SMD3225-4P
Connections:
- net +5v: now also C7.1

Commit message: - All footprints laid out; DRC NOT run yet, likely has many violations - Thin out peripheral headers, move remaining to dispersed test pads - Update kicad-libraries
Parts:
- removed TP5: TestPoint, TestPoint:TestPoint_Pad_2.0x2.0mm, symbol Connector:TestPoint
- added C4, C7: 10uF, Capacitor_SMD:C_0805_2012Metric, symbol Device:C_Small
- renumbered C7 to C3
Connections:
- net +5v: now also C4.1
- net GND: now also C4.2, C7.2
- net M2_3v3: now also C7.1; no longer C3.1
Changed lines of the file:
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@@
-	)
-	(junction
-		(at 240.03 71.12)
-		(diameter 0)
-		(color 0 0 0 0)
 	)
 	(junction
@@
 	(wire
 		(pts
-			(xy 240.03 71.12) (xy 240.03 76.2)
+			(xy 240.03 68.58) (xy 240.03 76.2)
 		)
 		(stroke
@@
 	(wire
 		(pts
-			(xy 240.03 71.12) (xy 240.03 68.58)
-		)
-		(stroke
-			(width 0)
-			(type solid)
-		)
-	)
-	(wire
-		(pts
 			(xy 193.04 24.13) (xy 195.58 24.13)
 		)
@@
 			(width 0)
 			(type default)
-		)
-	)
-	(wire
-		(pts
-			(xy 240.03 71.12) (xy 246.38 71.12)
-		)
-		(stroke
-			(width 0)
-			(type solid)
 		)
 	)
@@
 					(unit 1)
 				)
-			)
-		)
-	)
-	(symbol
-		(lib_id "Connector:TestPoint")
-		(at 246.38 71.12 270)
-		(unit 1)
-		(exclude_from_sim no)
-		(in_bom no)
-		(on_board yes)
-		(dnp yes)
-		(property "Reference" "TP5"
-			(at 247.65 74.93 90)
-			(effects
-				(font
-					(size 1.27 1.27)
-				)
-				(justify left)
-			)
-		)
-		(property "Value" "TestPoint"
-			(at 245.11 73.025 90)
-			(effects
-				(font
-					(size 1.27 1.27)
-				)
-				(justify left)
-			)
-		)
-		(property "Footprint" "TestPoint:TestPoint_Pad_2.0x2.0mm"
-			(at 246.38 76.2 0)
-			(effects
-				(font
-					(size 1.27 1.27)
-				)
-				(hide yes)
-			)
-		)
-		(property "Datasheet" "~"
-			(at 246.38 76.2 0)
-			(effects
-				(font
-					(size 1.27 1.27)
-				)
-				(hide yes)
-			)
-		)
-		(property "Description" "test point"
-			(at 246.38 71.12 0)
-			(effects
-				(font
-					(size 1.27 1.27)
-				)
-				(hide yes)
-			)
-		)
-		(property "Field4" "nf"
-			(at 246.38 71.12 0)
-			(effects
-				(font
-					(size 1.27 1.27)
-				)
-				(hide yes)
-			)
-		)
-		(property "Field5" "nf"
-			(at 246.38 71.12 0)
-			(effects
-				(font
-					(size 1.27 1.27)
-				)
-				(hide yes)
-			)
-		)
-		(property "Field6" "nf"
-			(at 246.38 71.12 0)
-			(effects
-				(font
-					(size 1.27 1.27)
-				)
-				(hide yes)
-			)
-		)
-		(property "Field7" "nf"
-			(at 246.38 71.12 0)
-			(effects
-				(font
-					(size 1.27 1.27)
-				)
-				(hide yes)
-			)
-		)
-		(property "Part Description" "Test point"
-			(at 246.38 71.12 0)
-			(effects
-				(font
-					(size 1.27 1.27)
-				)
-				(hide yes)
-			)
-		)
-		(property "Class" ""
-			(at 246.38 71.12 90)
-			(effects
-				(font
-					(size 1.27 1.27)
-				)
-				(hide yes)
-			)
-		)
-		(property "Dielectric_Class" ""
-			(at 246.38 71.12 90)
-			(effects
-				(font
-					(size 1.27 1.27)
-				)
-				(hide yes)
-			)
-		)
-		(property "Color" ""
-			(at 246.38 71.12 90)
-			(effects
-				(font
-					(size 1.27 1.27)
-				)
-				(hide yes)
-			)
-		)
-		(pin "1"
-		)
-		(instances
-			(project "garden_guard"
-				(path "/dcdac9d4-ef08-426f-b97c-7b9219501e71/5751e26b-0975-4f8f-84d7-7785f65d80bc"
-					(reference "TP5")
-					(unit 1)
-				)
