File: projects/garden_guard/Peripherals.kicad_sch (KiCad schematic)
At the start: 12 parts, among them J10 Conn_02x01, J11 Conn_02x01, J8 Conn_02x05_Odd_Even, J9 Conn_02x06_Odd_Even, U12 DMN2028USS-13, U13 DMN2028USS-13

Commit message: JLC part audit - Power - Peripherals - Replace ETQ-P4M2R2KFM with SPM6550T-2R2M-HZ
Parts:
- D6: Class (none) -> diode; Critical (none) -> no; JLCPCB_PN (none) -> C8678; MPN (none) -> SS34; Mfr (none) -> MDD
- R24, R26: Class (none) -> resistor; Critical (none) -> no; JLCPCB_PN (none) -> C105588; Package (none) -> 0603; Voltage (none) -> 75V
- R25, R27: Class (none) -> resistor; Critical (none) -> no; JLCPCB_PN (none) -> C14675; Package (none) -> 0603; Power (none) -> 1/10W; Voltage (none) -> 75V
- U12, U13: Class (none) -> mosfet; Critical (none) -> review; JLCPCB_PN (none) -> C5157769; Package (none) -> SO-8

Commit message: - All footprints laid out; DRC NOT run yet, likely has many violations - Thin out peripheral headers, move remaining to dispersed test pads - Update kicad-libraries
Parts:
- J8: footprint Connector_PinHeader_2.54mm:PinHeader_2x05_P2.54mm_Vertical -> Connector_PinHeader_2.54mm:PinHeader_2x05_P2.54mm_Vertical_SMD
- J9: footprint Connector_PinHeader_2.54mm:PinHeader_2x06_P2.54mm_Vertical -> Connector_PinHeader_2.54mm:PinHeader_2x06_P2.54mm_Vertical_SMD
Changed lines of the file:
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@@
 		(exclude_from_sim no)
 		(in_bom no)
-		(on_board yes)
+		(on_board no)
 		(dnp yes)
 		(property "Reference" "J9"
@@
 			)
 		)
-		(property "Footprint" "Connector_PinHeader_2.54mm:PinHeader_2x06_P2.54mm_Vertical"
+		(property "Footprint" "Connector_PinHeader_2.54mm:PinHeader_2x06_P2.54mm_Vertical_SMD"
 			(at 118.11 48.26 0)
 			(effects
@@
 		(exclude_from_sim no)
 		(in_bom no)
-		(on_board yes)
+		(on_board no)
 		(dnp yes)
 		(fields_autoplaced yes)
@@
 			)
 		)
-		(property "Footprint" "Connector_PinHeader_2.54mm:PinHeader_2x05_P2.54mm_Vertical"
+		(property "Footprint" "Connector_PinHeader_2.54mm:PinHeader_2x05_P2.54mm_Vertical_SMD"
 			(at 57.15 45.72 0)
 			(effects
